File: Mic Pre-Amp.sch (KiCad schematic (older format))
At the start: 16 parts, among them J1 AudioPlug3, J2 AudioJack3, Q1 BC337

Commit message: v2.1 | Op-Amp Based | Working | have 20KHz noice, Source of noise unknown, Clipping Happens at low frequencies (100Hz)
Parts:
- removed C1, C2: 100u, symbol Device:CP
- removed C3: 470u, symbol Device:CP
- removed J1: AudioPlug3, symbol Connector:AudioPlug3
- removed Q1: BC337, Package_TO_SOT_THT:TO-92_Inline, symbol Transistor_BJT:BC337
- removed R1: 8.2k, symbol Device:R
- removed R2: 3.3k, symbol Device:R
- removed R3: R, symbol Device:R
- removed R4: 330, symbol Device:R
- removed R5: 5k, symbol Device:R
- removed RV1: 20k, symbol Device:R_POT
- added C101: 220u, Capacitor_THT:CP_Radial_D10.0mm_P2.50mm, symbol Device:CP
- added C102: 220u, Capacitor_THT:CP_Radial_D10.0mm_P2.50mm_P5.00mm, symbol Device:CP
- added J101: AudioPlug3, symbol Connector:AudioPlug3
- added R101, R106, R107: 1k, Resistor_THT:R_Axial_DIN0207_L6.3mm_D2.5mm_P7.62mm_Horizontal, symbol Device:R
- added R102: 20k, Resistor_THT:R_Axial_DIN0207_L6.3mm_D2.5mm_P7.62mm_Horizontal, symbol Device:R
- added R103: R, Resistor_THT:R_Axial_DIN0207_L6.3mm_D2.5mm_P7.62mm_Horizontal, symbol Device:R
- added R104, R105: 100k, Resistor_THT:R_Axial_DIN0207_L6.3mm_D2.5mm_P7.62mm_Horizontal, symbol Device:R
- added R108: 10k, Resistor_THT:R_Axial_DIN0207_L6.3mm_D2.5mm_P7.62mm_Horizontal, symbol Device:R
- added U101: TL072, Package_DIP:DIP-8_W7.62mm, symbol Amplifier_Operational:TL072
Connections:
- net labels added: GNDREF
- wire segments 26 -> 24
Other:
- moved on the sheet: C4, MK1, R6, RV2
